File: LoRa_Node_Schematic.sch (EAGLE design)
At the start: 0 parts

Commit message: done
Parts:
- added U1: ATSAMD21G18A-AU, ATSAMD21G18A_AU:ATSAMD21G18A-AU
- added U2: RFM95W-915S2, RFM95W-915S2:RFM95W-915S2
Changed lines of the file:
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@@
 <part name="FRAME1" library="frames" library_urn="urn:adsk.eagle:library:229" deviceset="A4L-LOC" device=""/>
 <part name="FRAME2" library="frames" library_urn="urn:adsk.eagle:library:229" deviceset="A4L-LOC" device=""/>
+<part name="U1" library="ATSAMD21G18A_AU" deviceset="ATSAMD21G18A-AU" device=""/>
+<part name="U2" library="RFM95W-915S2" deviceset="RFM95W-915S2" device=""/>
 </parts>
 <sheets>
@@
 <attribute name="LAST_DATE_TIME" x="217.17" y="10.16" size="2.286" layer="94"/>
 <attribute name="SHEET" x="230.505" y="5.08" size="2.54" layer="94"/>
+</instance>
+<instance part="U1" gate="A" x="73.66" y="91.44" smashed="yes">
+<attribute name="NAME" x="73.66" y="135.89" size="2.0828" layer="95" ratio="6" rot="SR0" align="bottom-center"/>
+<attribute name="VALUE" x="73.66" y="45.72" size="2.0828" layer="96" ratio="6" rot="SR0" align="bottom-center"/>
+</instance>
+<instance part="U2" gate="G$1" x="187.96" y="119.38" smashed="yes">
+<attribute name="NAME" x="187.96" y="135.89" size="1.778" layer="95" align="bottom-center"/>
+<attribute name="VALUE" x="187.96" y="101.6" size="1.778" layer="96" align="bottom-center"/>
 </instance>
 </instances>
@@
 <attribute name="SHEET" x="230.505" y="5.08" size="2.54" layer="94"/>
 </instance>
+<instance part="U1" gate="B" x="215.9" y="132.08" smashed="yes">
+<attribute name="NAME" x="215.9" y="151.13" size="2.0828" layer="95" ratio="6" rot="SR0" align="bottom-center"/>
+<attribute name="VALUE" x="215.9" y="111.76" size="2.0828" layer="96" ratio="6" rot="SR0" align="bottom-center"/>
+</instance>
 </instances>

Commit message: update
Parts:
- added J1: ZX62D-B-5PA8, ZX62D-B-5PA8:ZX62D-B-5PA8
- added U3: AP2112K-3.3, AP2112K-3.3:AP2112K-3.3
- added U4: MCP73831-2ACI/OT, MCP73831-2ACI_OT:MCP73831-2ACI/OT
Changed lines of the file:
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@@
 <part name="U1" library="ATSAMD21G18A_AU" deviceset="ATSAMD21G18A-AU" device=""/>
 <part name="U2" library="RFM95W-915S2" deviceset="RFM95W-915S2" device=""/>
+<part name="U3" library="AP2112K-3.3" deviceset="AP2112K-3.3" device=""/>
+<part name="U4" library="MCP73831-2ACI_OT" deviceset="MCP73831-2ACI/OT" device=""/>
+<part name="J1" library="ZX62D-B-5PA8" deviceset="ZX62D-B-5PA8" device=""/>
 </parts>
 <sheets>
@@
 <attribute name="VALUE" x="215.9" y="111.76" size="2.0828" layer="96" ratio="6" rot="SR0" align="bottom-center"/>
 </instance>
+<instance part="U3" gate="G$1" x="83.82" y="132.08" smashed="yes">
+<attribute name="NAME" x="83.82" y="140.97" size="2.08946875" layer="95" ratio="10" rot="SR0" align="bottom-center"/>
+<attribute name="VALUE" x="83.82" y="121.92" size="2.0883" layer="96" ratio="10" rot="SR0" align="bottom-center"/>
+</instance>
+<instance part="U4" gate="G$1" x="68.58" y="83.82" smashed="yes">
+<attribute name="NAME" x="68.58" y="92.71" size="2.08681875" layer="95" ratio="10" rot="SR0" align="bottom-center"/>
+<attribute name="VALUE" x="68.58" y="68.58" size="2.085940625" layer="96" ratio="10" rot="SR0" align="bottom-center"/>
+</instance>
+<instance part="J1" gate="G$1" x="27.94" y="142.24" smashed="yes">
+<attribute name="NAME" x="27.94" y="153.67" size="1.77961875" layer="95" align="bottom-center"/>
+<attribute name="VALUE" x="27.94" y="129.54" size="1.778109375" layer="96" align="bottom-center"/>
+</instance>
 </instances>
