File: LoRa_Node_Schematic.sch (EAGLE design)
At the start: 5 parts, among them J1 ZX62D-B-5PA8, U1 ATSAMD21G18A-AU, U2 RFM95W-915S2, U3 AP2112K-3.3, U4 MCP73831-2ACI/OT

Commit message: update 27.12
Parts:
- added C1, C2: 20p, rcl:C-EUC0402
- added C3: 4n7, rcl:C-EUC0805
- added C4: 100n, rcl:C-EUC0402
- added J2: S2B-PH-SM4-TB(LF)(SN), S2B-PH-SM4-TB_LF_SN:S2B-PH-SM4-TB(LF)(SN)
- added R1: 1M, rcl:R-EU_R0402
- added R2: 10k, rcl:R-EU_R0402
- added R3: 330, rcl:R-EU_R0402
- added S1: KMR231NGLFS, KMR231NGLFS:KMR231NGLFS
- added TP1, TP2: TPTP10R, testpad:TPTP10R
- added U5: SHT40-AD1B-R2, SHT40-AD1B-R2:SHT40-AD1B-R2
- added Y1: 32.768KHZ, ABS07-32.768KHZ-T:ABS07-32.768KHZ-T
Connections:
- new net +3V3: R2.2
- new net A0: U1A.PA02/A0
- new net A1: U1A.PB08/A1
- new net A2: U1A.PB09/A2
- new net A3: U1A.PA04/A3
- new net A4: U1A.PA05/A4
- new net A5: U1A.PB02/A5
- new net AREF: U1A.PA03/AREF
- new net CS_LORA: U1A.PA06/D8/CS_LORA, U2.NSS
- new net D0: U1A.PA11/D0
- new net D1: U1A.PA10/D1
- new net D10: U1A.PA18/D10
- new net D2: U1A.PA14/D2
- new net D5: U1A.PA15/D5
- new net D6: U1A.PA20/D6
- new net D7: U1A.PA21/D7
- new net D9: U1A.PA07/D9
- new net GND: C1.1, C2.1, C3.2, C4.2, J1.GND, R1.1, S1.NO, U1A.EPAD, U2.GND
- new net I2C_SCL: U1A.PA23/SCL, U5.SCL
- new net I2C_SDA: U1A.PA22/SDA, U5.SDA
- new net IRQ_LORA: U1A.PA09/D3/DIO0_IRQ_LORA, U2.DIO0
- new net MISO_LORA: U1A.PA12/MISO_LORA, U2.MISO
- new net MOSI_LORA: U1A.PB10/MOSI_LORA, U2.MOSI
- new net N$1: C3.1, J1.SHIELD, R1.2
- new net N$2: C1.2, U1A.PA00/XIN32, Y1.2
- new net N$3: C2.2, U1A.PA01/XOUT32, Y1.1
- new net N$4: R3.2, S1.COM
- new net RESETN: C4.1, R2.1, R3.1, U1A.!RESET
- new net RST_LORA: U1A.PA08/D4/RST_LORA, U2.RESET
- new net SCK_LORA: U1A.PB11/SCK_LORA, U2.SCK
- new net SPI_MISO: U1A.PA19/D12/MISO
- new net SPI_MOSI: U1A.PA16/D11/MOSI
- new net SPI_SCK: U1A.PA17/D13/SCK
- new net SWCLK: TP1.TP, U1A.PA30/SWCLK
- new net SWDIO: TP2.TP, U1A.PA31/SWDIO
- new net USB_D+: J1.D+, U1A.PA24/USB_D-
- new net USB_D-: J1.D-, U1A.PA25/USB_D+
- new net VBUS: J1.VBUS
Other:
- note added: "N/C"
- moved on the sheet: U1A

Commit message: update29.12
Parts:
- added C5: 100n, rcl:C-EUC0402
- added D1: PRTR5V0U2X,215, PRTR5V0U2X_215:PRTR5V0U2X,215
- added R4, R5: 10k, rcl:R-EU_R0402
Connections:
- net +3V3: now also C5.1, R4.2, R5.2, U5.VDD
- net GND: now also C5.2, U5.VSS
- net I2C_SCL: now also R5.1
- net I2C_SDA: now also R4.1
- net N$1: now also D1.P$1
- net USB_D+: now also D1.P$2
- net USB_D-: now also D1.P$3
- net VBUS: now also D1.P$4
Other:
- moved on the sheet: C3, R1, U2, U3, U5

Commit message: update
Parts:
- added C10: 1µ, rcl:C-EUC0402
- added C11, C6, C7, C8, C9: 100n, rcl:C-EUC0402
- added C12: 4u7, rcl:C-EUC0603
- added C13, C14: 1u, rcl:C-EUC0402
- added C15: 10u, rcl:C-EUC0603
- added D2: MBR120VLSFT1G, MBR120VLSFT1G:MBR120VLSFT1G
- added L1: BLM18PG471SN1D, BLM18PG471SN1D:BLM18PG471SN1D
- added R6: 100k, rcl:R-EU_R0402
- R3: value 330 -> 330R
Connections:
- new net N$5: C10.1, U1B.VDDCORE
- new net N$6: C11.1, C12.1, L1.2, U1B.VDDANA
- new net N$7: R6.2, U3.EN
- new net VBAT: D2.12
- net +3V3: now also C14.1, C6.1, C7.1, C8.1, C9.1, L1.1, U1B.VDDIN, U1B.VDDIO, U1B.VDDIO_2, U2.3.3V, U3.VOUT
- net GND: now also C10.2, C11.2, C12.2, C13.2, C14.2, C15.2, C6.2, C7.2, C8.2, C9.2, U1B.GND, U1B.GNDANA, U1B.GND_2, U1B.GND_3, U3.GND
- net VBUS: now also C13.1, C15.1, D2.11, R6.1, U3.VIN
Other:
- moved on the sheet: J2, U1B, U3, U4

Commit message: Review Version
Parts:
- removed R2: 10k, rcl:R-EU_R0402
- added ANT1: 0868AT43A0020E, 0868AT43A0020E:0868AT43A0020E
- added C16, C17, C22: 4u7, rcl:C-EUC0603
- added C18: 3p9, rcl:C-EUC0402
- added C19: 0p3, rcl:C-EUC0402
- added C20: 10u, rcl:C-EUC0603
- added C21: 100n, rcl:C-EUC0402
- added JP1, JP2: (no value), pinhead:PINHD-1X12
- added L2: 18n, Inductor_SMD:INDUCTOR_0402_SMD
- added LED1: (no value), led:LEDCHIP-LED0805
- added R7: 10k, rcl:R-EU_R0402
- added R8: 1k, rcl:R-EU_R0402
- U2: value RFM95W-915S2 -> RFM95W-868S2; device RFM95W-915S2:RFM95W-915S2 -> RFM95W-868S2:RFM95W-868S2
Connections:
- new net N$10: LED1.C, R8.1
- new net N$11: ANT1.FEED, C19.1, L2.2
- new net N$12: C18.1, L2.1, U2.ANT
- new net N$8: R7.1, U4.PROG
- new net N$9: R8.2, U4.STAT
- net +3V3: now also C20.1, JP2.1; no longer R2.2
- net A0: now also JP2.2
- net A1: now also JP2.3
- net A2: now also JP2.4
- net A3: now also JP2.5
- net A4: now also JP2.6
- net A5: now also JP2.7
- net AREF: now also C21.1, C22.1, JP2.8
- net D0: now also JP1.2
- net D1: now also JP1.3
- net D10: now also JP1.9
- net D2: now also JP1.4
- net D5: now also JP1.5
- net D6: now also JP1.6
- net D7: now also JP1.7
- net D9: now also JP1.8
- net GND: now also C16.2, C17.2, C18.2, C19.2, C20.2, C21.2, C22.2, J2.2, J2.SHIELD, JP1.12, JP2.12, R7.2, U4.VSS
- net I2C_SCL: now also JP1.11
- net I2C_SDA: now also JP1.10
- net RESETN: no longer R2.1
- net SPI_MISO: now also JP2.11
- net SPI_MOSI: now also JP2.10
- net SPI_SCK: now also JP2.9
- net VBAT: now also C16.1, J2.1, U4.VBAT
- net VBUS: now also C17.1, JP1.1, LED1.A, U4.VDD
Other:
- moved on the sheet: C10, C11, C12, C13, C14, C15, C3, C4, C5, C6, C7, C8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

Commit message: update
Parts:
- removed J2: S2B-PH-SM4-TB(LF)(SN), S2B-PH-SM4-TB_LF_SN:S2B-PH-SM4-TB(LF)(SN)
- added J3: B2B-PH-K-S(LF)(SN), B2B-PH-K-S_LF_SN:B2B-PH-K-S(LF)(SN)
Connections:
- net N$1 renamed USB_SHIELD
- net N$10 renamed VBAT_STAT_R
- net N$11 renamed ANTENNA_L
- net N$12 renamed ANTENNA
- net N$2 renamed XIN32
- net N$3 renamed XOUT32
- net N$4 renamed RESETN_R
- net N$5 renamed VDDCORE
- net N$6 renamed VDDANA
- net N$7 renamed 3V3_EN
- net N$8 renamed VBAT_PROG
- net N$9 renamed VBAT_STAT
- removed net USB_D+: D1.P$2, J1.D+, U1A.PA24/USB_D-
- removed net USB_D-: D1.P$3, J1.D-, U1A.PA25/USB_D+
- new net USB_D_N: D1.P$3, J1.D-, U1A.PA24/USB_D-
- new net USB_D_P: D1.P$2, J1.D+, U1A.PA25/USB_D+
- net GND: now also J3.2; no longer J2.2, J2.SHIELD
- net VBAT: now also J3.1; no longer J2.1
Changed lines of the file:
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@@
 <setting verticaltext="up"/>
 </settings>
-<grid distance="0.1" unitdist="inch" unit="inch" style="lines" multiple="1" display="yes" altdistance="0.05" altunitdist="inch" altunit="inch"/>
+<grid distance="0.1" unitdist="inch" unit="inch" style="lines" multiple="1" display="no" altdistance="0.01" altunitdist="inch" altunit="inch"/>
 <layers>
 <layer number="1" name="Top" color="4" fill="1" visible="no" active="no"/>
@@
 </variantdefs>
 <classes>
-<class number="0" name="default" width="0" drill="0">
+<class number="0" name="default" width="0.23" drill="0">
+<clearance class="0" value="0.254"/>
+</class>
+<class number="1" name="Power" width="0.254" drill="0">
+<clearance class="0" value="0.254"/>
+<clearance class="1" value="0.254"/>
+</class>
+<class number="2" name="Diff" width="0.165" drill="0">
+<clearance class="0" value="0.5"/>
+<clearance class="1" value="0.5"/>
+<clearance class="2" value="0.18"/>
+</class>
+<class number="3" name="Antenna" width="0.21" drill="0">
+<clearance class="0" value="0.5"/>
+<clearance class="1" value="0.2"/>
+<clearance class="2" value="0.5"/>
+<clearance class="3" value="0.5"/>
 </class>
 </classes>
@@
 <part name="GND7" library="supply1" library_urn="urn:adsk.eagle:library:371" deviceset="GND" device=""/>
 <part name="R3" library="rcl" library_urn="urn:adsk.eagle:library:334" deviceset="R-EU_" device="R0402" package3d_urn="urn:adsk.eagle:package:23547/3" value="330R"/>
-<part name="J2" library="S2B-PH-SM4-TB_LF_SN" deviceset="S2B-PH-SM4-TB(LF)(SN)" device=""/>
 <part name="D1" library="PRTR5V0U2X_215" deviceset="PRTR5V0U2X,215" device=""/>
 <part name="R4" library="rcl" library_urn="urn:adsk.eagle:library:334" deviceset="R-EU_" device="R0402" package3d_urn="urn:adsk.eagle:package:23547/3" value="10k"/>
@@
 <part name="GND26" library="supply1" library_urn="urn:adsk.eagle:library:371" deviceset="GND" device=""/>
 <part name="GND27" library="supply1" library_urn="urn:adsk.eagle:library:371" deviceset="GND" device=""/>
+<part name="J3" library="B2B-PH-K-S_LF_SN" deviceset="B2B-PH-K-S(LF)(SN)" device=""/>
 </parts>
 <sheets>
@@
 </segment>
 </net>
-<net name="GND" class="0">
+<net name="GND" class="1">
 <segment>
 <pinref part="U1" gate="A" pin="EPAD"/>
@@
 </segment>
 </net>
-<net name="N$2" class="0">
+<net name="XIN32" class="0">
 <segment>
 <pinref part="U1" gate="A" pin="PA00/XIN32"/>
@@
 </segment>
 </net>
-<net name="N$3" class="0">
+<net name="XOUT32" class="0">
 <segment>
 <pinref part="U1" gate="A" pin="PA01/XOUT32"/>
@@
 </segment>
 </net>
-<net name="USB_D+" class="0">
-<segment>
-<pinref part="U1" gate="A" pin="PA24/USB_D-"/>
-<wire x1="58.42" y1="121.92" x2="43.18" y2="121.92" width="0.1524" layer="91"/>
-<label x="43.18" y="121.92" size="1.778" layer="95"/>
-</segment>
-</net>
-<net name="USB_D-" class="0">
-<segment>
-<pinref part="U1" gate="A" pin="PA25/USB_D+"/>
-<wire x1="58.42" y1="119.38" x2="43.18" y2="119.38" width="0.1524" layer="91"/>
-<label x="43.18" y="119.38" size="1.778" layer="95"/>
-</segment>
-</net>
 <net name="SWCLK" class="0">
 <segment>
@@
 </segment>
 </net>
-<net name="N$4" class="0">
+<net name="RESETN_R" class="0">
 <segment>
 <pinref part="S1" gate="G$1" pin="COM"/>
@@
 </segment>
 </net>
-<net name="+3V3" class="0">
+<net name="+3V3" class="1">
 <segment>
 <pinref part="U5" gate="A" pin="VDD"/>
@@
 </segment>
 </net>
-<net name="N$11" class="0">
+<net name="ANTENNA_L" class="3">
 <segment>
 <pinref part="L2" gate="G$1" pin="2"/>
@@
 </segment>
 </net>
-<net name="N$12" class="0">
+<net name="ANTENNA" class="3">
 <segment>
 <pinref part="L2" gate="G$1" pin="1"/>
@@
 <wire x1="160.02" y1="106.68" x2="175.26" y2="106.68" width="0.1524" layer="91"/>
 <junction x="175.26" y="106.68"/>
+</segment>
+</net>
+<net name="USB_D_P" class="2">
+<segment>
+<wire x1="58.42" y1="119.38" x2="43.18" y2="119.38" width="0.1524" layer="91"/>
+<pinref part="U1" gate="A" pin="PA25/USB_D+"/>
+<label x="43.18" y="119.38" size="1.778" layer="95"/>
+</segment>
+</net>
+<net name="USB_D_N" class="2">
+<segment>
+<wire x1="58.42" y1="121.92" x2="43.18" y2="121.92" width="0.1524" layer="91"/>
+<pinref part="U1" gate="A" pin="PA24/USB_D-"/>
+<label x="43.18" y="121.92" size="1.778" layer="95"/>
 </segment>
 </net>
@@
 <attribute name="VALUE" x="66.548" y="124.46" size="1.778" layer="96" rot="R90" align="bottom-center"/>
 </instance>
-<instance part="J2" gate="G$1" x="203.2" y="43.18" smashed="yes">
-<attribute name="NAME" x="203.2" y="49.53" size="1.778" layer="95" align="bottom-center"/>
-<attribute name="VALUE" x="203.2" y="35.56" size="1.778" layer="96" align="bottom-center"/>
-</instance>
 <instance part="D1" gate="G$1" x="83.82" y="142.24" smashed="yes">
 <attribute name="NAME" x="81.27258125" y="134.699640625" size="1.7832" layer="95"/>
@@
 <instance part="GND27" gate="1" x="177.8" y="127" smashed="yes">
 <attribute name="VALUE" x="175.26" y="124.46" size="1.778" layer="96"/>
+</instance>
+<instance part="J3" gate="G$1" x="200.66" y="45.72" smashed="yes">
+<attribute name="NAME" x="200.655640625" y="49.022" size="1.778" layer="95" align="bottom-center"/>
+<attribute name="VALUE" x="200.655409375" y="38.1" size="1.778" layer="96" align="bottom-center"/>
 </instance>
 </instances>
@@
 </busses>
 <nets>
-<net name="USB_D+" class="0">
+<net name="USB_D_P" class="2">
 <segment>
 <wire x1="106.68" y1="152.4" x2="86.36" y2="152.4" width="0.1524" layer="91"/>
@@
 </segment>
 </net>
-<net name="USB_D-" class="0">
+<net name="USB_D_N" class="2">
 <segment>
 <wire x1="106.68" y1="154.94" x2="91.44" y2="154.94" width="0.1524" layer="91"/>
@@
 </segment>
 </net>
-<net name="VBUS" class="0">
+<net name="VBUS" class="1">
 <segment>
 <pinref part="J1" gate="G$1" pin="VBUS"/>
@@
 </segment>
 </net>
-<net name="GND" class="0">
+<net name="GND" class="1">
 <segment>
 <pinref part="J1" gate="G$1" pin="GND"/>
@@
 </segment>
 <segment>
-<pinref part="J2" gate="G$1" pin="2"/>
 <wire x1="193.04" y1="43.18" x2="185.42" y2="43.18" width="0.1524" layer="91"/>
-<wire x1="185.42" y1="43.18" x2="185.42" y2="40.64" width="0.1524" layer="91"/>
-<pinref part="J2" gate="G$1" pin="SHIELD"/>
-<wire x1="185.42" y1="40.64" x2="185.42" y2="35.56" width="0.1524" layer="91"/>
-<wire x1="193.04" y1="40.64" x2="185.42" y2="40.64" width="0.1524" layer="91"/>
-<junction x="185.42" y="40.64"/>
+<wire x1="185.42" y1="43.18" x2="185.42" y2="35.56" width="0.1524" layer="91"/>
 <pinref part="GND18" gate="1" pin="GND"/>
+<pinref part="J3" gate="G$1" pin="2"/>
 </segment>
 <segment>
@@
 </segment>
 </net>
-<net name="N$1" class="0">
+<net name="USB_SHIELD" class="0">
 <segment>
 <pinref part="J1" gate="G$1" pin="SHIELD"/>
@@
 </segment>
 </net>
-<net name="N$5" class="0">
+<net name="VDDCORE" class="1">
 <segment>
 <pinref part="C10" gate="G$1" pin="1"/>
@@
 </segment>
 </net>
-<net name="N$6" class="0">
+<net name="VDDANA" class="1">
 <segment>
 <pinref part="U1" gate="B" pin="VDDANA"/>
@@
 </segment>
 </net>
-<net name="N$7" class="0">
+<net name="3V3_EN" class="0">
 <segment>
 <pinref part="U3" gate="G$1" pin="EN"/>
@@
 </segment>
 </net>
-<net name="VBAT" class="0">
+<net name="VBAT" class="1">
 <segment>
 <pinref part="D2" gate="G$1" pin="12"/>
@@
 </segment>
 <segment>
-<pinref part="J2" gate="G$1" pin="1"/>
 <wire x1="193.04" y1="45.72" x2="185.42" y2="45.72" width="0.1524" layer="91"/>
 <wire x1="185.42" y1="45.72" x2="185.42" y2="53.34" width="0.1524" layer="91"/>
 <pinref part="V12" gate="G$1" pin="VBAT"/>
-</segment>
-</net>
-<net name="N$8" class="0">
+<pinref part="J3" gate="G$1" pin="1"/>
+</segment>
+</net>
+<net name="VBAT_PROG" class="0">
 <segment>
 <pinref part="U4" gate="G$1" pin="PROG"/>
@@
 </segment>
 </net>
-<net name="N$9" class="0">
+<net name="VBAT_STAT" class="0">
 <segment>
 <pinref part="R8" gate="G$1" pin="2"/>
@@
 </segment>
 </net>
-<net name="N$10" class="0">
+<net name="VBAT_STAT_R" class="0">
 <segment>
 <pinref part="LED1" gate="G$1" pin="C"/>
@@
 </segment>
 </net>
-<net name="+3V3" class="0">
+<net name="+3V3" class="1">
 <segment>
 <pinref part="C7" gate="G$1" pin="1"/>

Commit message: update
Parts:
- added H1, H2, H3, H4: MOUNT-HOLE2.5, Adafruit Feather M0 RFMxx:MOUNT-HOLE2.5
- JP1, JP2: device pinhead:PINHD-1X12 -> adafruit:PINHD-1X12-CB
- U2: value RFM95W-868S2 -> RFM95W-868S2SMALL; device RFM95W-868S2:RFM95W-868S2 -> RFM95W-868S2:RFM95W-868S2SMALL
