File: LoRa_Node_Schematic.sch (EAGLE design)
At the start: 52 parts, among them J1 ZX62D-B-5PA8, J3 B2B-PH-K-S(LF)(SN), U1 ATSAMD21G18A-AU, U2 RFM95W-868S2SMALL, U3 AP2112K-3.3, U4 MCP73831-2ACI/OT, U5 SHT40-AD1B-R2, Y1 32.768KHZ

Commit message: update
Connections:
- net A0: now also JP2.5; no longer JP2.2
- net A1: now also JP2.6; no longer JP2.3
- net A2: now also JP2.7; no longer JP2.4
- net A3: now also JP2.8; no longer JP2.5
- net A4: now also JP2.9; no longer JP2.6
- net A5: now also JP2.10; no longer JP2.7
- net AREF: now also JP2.11; no longer JP2.8
- net GND: no longer U1A.EPAD
- net SPI_MISO: now also JP2.2; no longer JP2.11
- net SPI_MOSI: now also JP2.4; no longer JP2.10
- net SPI_SCK: now also JP2.3; no longer JP2.9
Changed lines of the file:
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@@
 <classes>
 <class number="0" name="default" width="0.23" drill="0.2">
-<clearance class="0" value="0.254"/>
+<clearance class="0" value="0.2032"/>
 </class>
 <class number="1" name="Power" width="0.254" drill="0.2">
-<clearance class="0" value="0.254"/>
-<clearance class="1" value="0.254"/>
+<clearance class="0" value="0.2032"/>
+<clearance class="1" value="0.2032"/>
 </class>
 <class number="2" name="Diff" width="0.165" drill="0.2">
-<clearance class="0" value="0.254"/>
-<clearance class="1" value="0.254"/>
+<clearance class="0" value="0.2032"/>
+<clearance class="1" value="0.2032"/>
 <clearance class="2" value="0.18"/>
 </class>
@@
 <part name="J1" library="ZX62D-B-5PA8" deviceset="ZX62D-B-5PA8" device=""/>
 <part name="U5" library="SHT40-AD1B-R2" deviceset="SHT40-AD1B-R2" device=""/>
-<part name="GND1" library="supply1" library_urn="urn:adsk.eagle:library:371" deviceset="GND" device=""/>
 <part name="GND2" library="supply1" library_urn="urn:adsk.eagle:library:371" deviceset="GND" device=""/>
 <part name="Y1" library="ABS07-32.768KHZ-T" deviceset="ABS07-32.768KHZ-T" device="" value="32.768KHZ"/>
@@
 <attribute name="VALUE" x="203.2" y="40.64" size="2.0828" layer="96" ratio="6" rot="SR0" align="bottom-center"/>
 </instance>
-<instance part="GND1" gate="1" x="40.64" y="139.7" smashed="yes" rot="R270">
-<attribute name="VALUE" x="38.1" y="142.24" size="1.778" layer="96" rot="R270"/>
-</instance>
 <instance part="GND2" gate="1" x="233.68" y="121.92" smashed="yes">
 <attribute name="VALUE" x="231.14" y="119.38" size="1.778" layer="96"/>
@@
 </net>
 <net name="GND" class="1">
-<segment>
-<pinref part="U1" gate="A" pin="EPAD"/>
-<wire x1="58.42" y1="139.7" x2="43.18" y2="139.7" width="0.1524" layer="91"/>
-<pinref part="GND1" gate="1" pin="GND"/>
-</segment>
 <segment>
 <wire x1="210.82" y1="127" x2="233.68" y2="127" width="0.1524" layer="91"/>
@@
 <net name="SPI_SCK" class="0">
 <segment>
+<wire x1="81.28" y1="45.72" x2="96.52" y2="45.72" width="0.1524" layer="91"/>
+<label x="96.52" y="45.72" size="1.778" layer="95" align="bottom-right"/>
+<pinref part="JP2" gate="G$1" pin="3"/>
+</segment>
+</net>
+<net name="SPI_MOSI" class="0">
+<segment>
+<wire x1="81.28" y1="43.18" x2="96.52" y2="43.18" width="0.1524" layer="91"/>
+<label x="96.52" y="43.18" size="1.778" layer="95" align="bottom-right"/>
+<pinref part="JP2" gate="G$1" pin="4"/>
+</segment>
+</net>
+<net name="SPI_MISO" class="0">
+<segment>
+<wire x1="81.28" y1="48.26" x2="96.52" y2="48.26" width="0.1524" layer="91"/>
+<label x="96.52" y="48.26" size="1.778" layer="95" align="bottom-right"/>
+<pinref part="JP2" gate="G$1" pin="2"/>
+</segment>
+</net>
+<net name="I2C_SDA" class="0">
+<segment>
+<wire x1="50.8" y1="27.94" x2="66.04" y2="27.94" width="0.1524" layer="91"/>
+<label x="50.8" y="27.94" size="1.778" layer="95"/>
+<pinref part="JP1" gate="G$1" pin="10"/>
+</segment>
+</net>
+<net name="I2C_SCL" class="0">
+<segment>
+<wire x1="50.8" y1="25.4" x2="66.04" y2="25.4" width="0.1524" layer="91"/>
+<label x="50.8" y="25.4" size="1.778" layer="95"/>
+<pinref part="JP1" gate="G$1" pin="11"/>
+</segment>
+</net>
+<net name="A0" class="0">
+<segment>
+<wire x1="96.52" y1="40.64" x2="81.28" y2="40.64" width="0.1524" layer="91"/>
+<label x="96.52" y="40.64" size="1.778" layer="95" align="bottom-right"/>
+<pinref part="JP2" gate="G$1" pin="5"/>
+</segment>
+</net>
+<net name="A1" class="0">
+<segment>
+<wire x1="81.28" y1="38.1" x2="96.52" y2="38.1" width="0.1524" layer="91"/>
+<label x="96.52" y="38.1" size="1.778" layer="95" align="bottom-right"/>
+<pinref part="JP2" gate="G$1" pin="6"/>
+</segment>
+</net>
+<net name="A2" class="0">
+<segment>
+<wire x1="81.28" y1="35.56" x2="96.52" y2="35.56" width="0.1524" layer="91"/>
+<label x="96.52" y="35.56" size="1.778" layer="95" align="bottom-right"/>
+<pinref part="JP2" gate="G$1" pin="7"/>
+</segment>
+</net>
+<net name="A3" class="0">
+<segment>
+<wire x1="81.28" y1="33.02" x2="96.52" y2="33.02" width="0.1524" layer="91"/>
+<label x="96.52" y="33.02" size="1.778" layer="95" align="bottom-right"/>
+<pinref part="JP2" gate="G$1" pin="8"/>
+</segment>
+</net>
+<net name="A4" class="0">
+<segment>
 <wire x1="81.28" y1="30.48" x2="96.52" y2="30.48" width="0.1524" layer="91"/>
 <label x="96.52" y="30.48" size="1.778" layer="95" align="bottom-right"/>
@@
 </segment>
 </net>
-<net name="SPI_MOSI" class="0">
+<net name="A5" class="0">
 <segment>
 <wire x1="81.28" y1="27.94" x2="96.52" y2="27.94" width="0.1524" layer="91"/>
@@
 </segment>
 </net>
-<net name="SPI_MISO" class="0">
+<net name="AREF" class="0">
 <segment>
 <wire x1="81.28" y1="25.4" x2="96.52" y2="25.4" width="0.1524" layer="91"/>
@@
 </segment>
 </net>
-<net name="I2C_SDA" class="0">
-<segment>
-<wire x1="50.8" y1="27.94" x2="66.04" y2="27.94" width="0.1524" layer="91"/>
-<label x="50.8" y="27.94" size="1.778" layer="95"/>
-<pinref part="JP1" gate="G$1" pin="10"/>
-</segment>
-</net>
-<net name="I2C_SCL" class="0">
-<segment>
-<wire x1="50.8" y1="25.4" x2="66.04" y2="25.4" width="0.1524" layer="91"/>
-<label x="50.8" y="25.4" size="1.778" layer="95"/>
-<pinref part="JP1" gate="G$1" pin="11"/>
-</segment>
-</net>
-<net name="A0" class="0">
-<segment>
-<wire x1="96.52" y1="48.26" x2="81.28" y2="48.26" width="0.1524" layer="91"/>
-<label x="96.52" y="48.26" size="1.778" layer="95" align="bottom-right"/>
-<pinref part="JP2" gate="G$1" pin="2"/>
-</segment>
-</net>
-<net name="A1" class="0">
-<segment>
-<wire x1="81.28" y1="45.72" x2="96.52" y2="45.72" width="0.1524" layer="91"/>
-<label x="96.52" y="45.72" size="1.778" layer="95" align="bottom-right"/>
-<pinref part="JP2" gate="G$1" pin="3"/>
-</segment>
-</net>
-<net name="A2" class="0">
-<segment>
-<wire x1="81.28" y1="43.18" x2="96.52" y2="43.18" width="0.1524" layer="91"/>
-<label x="96.52" y="43.18" size="1.778" layer="95" align="bottom-right"/>
-<pinref part="JP2" gate="G$1" pin="4"/>
-</segment>
-</net>
-<net name="A3" class="0">
-<segment>
-<wire x1="81.28" y1="40.64" x2="96.52" y2="40.64" width="0.1524" layer="91"/>
-<label x="96.52" y="40.64" size="1.778" layer="95" align="bottom-right"/>
-<pinref part="JP2" gate="G$1" pin="5"/>
-</segment>
-</net>
-<net name="A4" class="0">
-<segment>
-<wire x1="81.28" y1="38.1" x2="96.52" y2="38.1" width="0.1524" layer="91"/>
-<label x="96.52" y="38.1" size="1.778" layer="95" align="bottom-right"/>
-<pinref part="JP2" gate="G$1" pin="6"/>
-</segment>
-</net>
-<net name="A5" class="0">
-<segment>
-<wire x1="81.28" y1="35.56" x2="96.52" y2="35.56" width="0.1524" layer="91"/>
-<label x="96.52" y="35.56" size="1.778" layer="95" align="bottom-right"/>
-<pinref part="JP2" gate="G$1" pin="7"/>
-</segment>
-</net>
-<net name="AREF" class="0">
-<segment>
-<wire x1="81.28" y1="33.02" x2="96.52" y2="33.02" width="0.1524" layer="91"/>
-<label x="96.52" y="33.02" size="1.778" layer="95" align="bottom-right"/>
-<pinref part="JP2" gate="G$1" pin="8"/>
-</segment>
-</net>

Commit message: update
Parts:
- removed H3, H4: MOUNT-HOLE2.5, Adafruit Feather M0 RFMxx:MOUNT-HOLE2.5
Changed lines of the file:
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@@
 <part name="H1" library="Adafruit Feather M0 RFMxx" deviceset="MOUNT-HOLE2.5" device=""/>
 <part name="H2" library="Adafruit Feather M0 RFMxx" deviceset="MOUNT-HOLE2.5" device=""/>
-<part name="H3" library="Adafruit Feather M0 RFMxx" deviceset="MOUNT-HOLE2.5" device=""/>
-<part name="H4" library="Adafruit Feather M0 RFMxx" deviceset="MOUNT-HOLE2.5" device=""/>
 <part name="GND1" library="supply1" library_urn="urn:adsk.eagle:library:371" deviceset="GND" device=""/>
 </parts>
@@
 <text x="53.34" y="101.6" size="1.778" layer="97">N/C</text>
 <text x="53.34" y="99.06" size="1.778" layer="97">N/C</text>
-<text x="182.88" y="45.72" size="1.778" layer="97">N/C</text>
 <text x="213.36" y="144.78" size="1.778" layer="97">N/C</text>
 <text x="213.36" y="142.24" size="1.778" layer="97">N/C</text>
@@
 <attribute name="VALUE" x="134.112" y="38.1762" size="1.778" layer="96"/>
 </instance>
-<instance part="H3" gate="G$1" x="132.08" y="33.02" smashed="yes">
-<attribute name="NAME" x="134.112" y="33.6042" size="1.778" layer="95"/>
-<attribute name="VALUE" x="134.112" y="30.5562" size="1.778" layer="96"/>
-</instance>
-<instance part="H4" gate="G$1" x="132.08" y="25.4" smashed="yes">
-<attribute name="NAME" x="134.112" y="25.9842" size="1.778" layer="95"/>
-<attribute name="VALUE" x="134.112" y="22.9362" size="1.778" layer="96"/>
-</instance>
 <instance part="GND1" gate="1" x="106.68" y="73.66" smashed="yes">

Commit message: update
Parts:
- C10: value 1µ -> 1u
Changed lines of the file:
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@@
 <part name="C8" library="rcl" library_urn="urn:adsk.eagle:library:334" deviceset="C-EU" device="C0402" package3d_urn="urn:adsk.eagle:package:23626/2" value="100n"/>
 <part name="C9" library="rcl" library_urn="urn:adsk.eagle:library:334" deviceset="C-EU" device="C0402" package3d_urn="urn:adsk.eagle:package:23626/2" value="100n"/>
-<part name="C10" library="rcl" library_urn="urn:adsk.eagle:library:334" deviceset="C-EU" device="C0402" package3d_urn="urn:adsk.eagle:package:23626/2" value="1µ"/>
+<part name="C10" library="rcl" library_urn="urn:adsk.eagle:library:334" deviceset="C-EU" device="C0402" package3d_urn="urn:adsk.eagle:package:23626/2" value="1u"/>
 <part name="GND10" library="supply1" library_urn="urn:adsk.eagle:library:371" deviceset="GND" device=""/>
 <part name="C11" library="rcl" library_urn="urn:adsk.eagle:library:334" deviceset="C-EU" device="C0402" package3d_urn="urn:adsk.eagle:package:23626/2" value="100n"/>
