File: LoRa_Node_Schematic.brd (EAGLE design)
At the start: 51 x 23 mm, 52 parts, among them J1 ZX62D-B-5PA8, J3 B2B-PH-K-S(LF)(SN), U1 ATSAMD21G18A-AU, U2 RFM95W-868S2SMALL, U3 AP2112K-3.3, U4 MCP73831-2ACI/OT, U5 SHT40-AD1B-R2, Y1 32.768KHZ

Commit message: update
Parts:
- moved C19 122.9 mm to (40.1, 8.85), flipped to the bottom, turned to 270 degrees
- moved C18 115.6 mm to (36.8, 8.85), flipped to the bottom, turned to 270 degrees
- moved L2 91.5 mm to (38.5, 9.50), flipped to the bottom, turned to 180 degrees
- moved TP2 83.7 mm to (-23.8, -3.21)
- moved R6 82.2 mm to (7.34, 29.1)
- moved TP1 80.2 mm to (-26.4, -2.71)
- moved C6 75.1 mm to (32.0, 13.6), turned to 90 degrees
- moved C10 73.7 mm to (-30.3, -3.21), turned to 180 degrees
- moved C1 73.0 mm to (-9.36, 1.06)
- moved C2 72.9 mm to (-14.4, 1.16)
- moved C9 72.4 mm to (-30.3, -7.70), turned to 180 degrees
- moved R3 69.1 mm to (-51.8, -4.85)
- moved C21 67.7 mm to (-19.2, 6.60)
- moved C22 67.2 mm to (-16.0, 6.53)
- moved C4 66.4 mm to (-45.1, -5.40)
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Routing:
- net ANTENNA: track 0.00 -> 12.8 mm
- net +3V3: track 0.00 -> 4.08 mm, vias 0 -> 1
- net ANTENNA_L: track 0.00 -> 3.88 mm
- net GND: track 0.00 -> 2.22 mm, vias 0 -> 14
- added copper zone on layer 16, net GND
- added copper zone on layer 3, net GND

Commit message: update
Parts:
- moved R1 46.4 mm to (5.50, 4.40)
- moved C3 43.3 mm to (5.00, 6.00), turned to 180 degrees
- moved D1 41.8 mm to (8.00, 11.8)
- moved U1 39.6 mm to (20.4, 12.1)
Routing:
- net USB_SHIELD: track 0.00 -> 23.9 mm
- net GND: track 2.22 -> 7.43 mm, vias 14 -> 16
- net VBUS: track 0.00 -> 2.94 mm, vias 0 -> 1

Commit message: update
Parts:
- moved C14 96.2 mm to (12.5, 2.20), flipped to the bottom, turned to 270 degrees
- moved C13 88.8 mm to (6.90, 2.20), flipped to the bottom, turned to 270 degrees
- moved C20 81.8 mm to (10.9, 2.20), flipped to the bottom, turned to 270 degrees
- moved R8 76.8 mm to (2.90, 17.6), flipped to the bottom, turned to 180 degrees
- moved D2 76.0 mm to (6.00, 20.6), flipped to the bottom, turned to 90 degrees
- moved R7 74.7 mm to (6.20, 16.5), flipped to the bottom, turned to 90 degrees
- moved C15 72.9 mm to (8.50, 2.20), flipped to the bottom, turned to 270 degrees
- moved C17 67.4 mm to (12.3, 17.6), flipped to the bottom, turned to 180 degrees
- moved R3 64.9 mm to (12.7, 2.80), turned to 180 degrees
- moved C16 62.4 mm to (12.0, 19.6), flipped to the bottom, turned to 180 degrees
- moved C4 59.9 mm to (14.4, 2.15), turned to 270 degrees
- moved LED1 56.3 mm to (3.60, 17.3), turned to 90 degrees
- moved S1 55.7 mm to (8.50, 2.00)
- moved C5 51.6 mm to (26.0, 36.3)
- moved R4 51.6 mm to (12.1, 46.5)
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Routing:
- net GND: track 7.43 -> 31.5 mm, vias 16 -> 20
- net USB_D_N: track 0.00 -> 14.6 mm
- net USB_D_P: track 0.26 -> 14.6 mm
- net VBUS: track 2.94 -> 16.1 mm, vias 1 -> 3
- net VBAT: track 0.00 -> 7.56 mm
- net RESETN_R: track 0.00 -> 5.75 mm
- net +3V3: track 4.08 -> 8.68 mm, vias 1 -> 2
- net VBAT_PROG: track 0.00 -> 1.76 mm
- net 3V3_EN: track 0.00 -> 1.67 mm
- net RESETN: track 0.00 -> 1.20 mm
- net USB_SHIELD: vias 0 -> 2

Commit message: update
Parts:
- moved U5 67.6 mm to (30.3, 30.4)
- moved C22 54.3 mm to (38.2, 4.65), turned to 90 degrees
- moved C12 51.5 mm to (27.6, 16.9), turned to 90 degrees
- moved C8 50.4 mm to (10.2, 8.75), turned to 180 degrees
- moved C7 49.7 mm to (18.1, 18.5), turned to 180 degrees
- moved C9 49.2 mm to (17.5, 3.80)
- moved C10 47.9 mm to (16.8, 5.20)
- moved TP1 46.9 mm to (20.1, 4.00)
- moved L1 46.6 mm to (29.2, 16.9), turned to 270 degrees
- moved C11 46.6 mm to (26.4, 11.3)
- moved TP2 46.0 mm to (21.6, 4.00)
- moved C21 45.8 mm to (26.4, 10.2)
- moved Y1 44.6 mm to (25.8, 6.30), turned to 270 degrees
- moved C2 43.4 mm to (28.5, 7.55), turned to 180 degrees
- moved C1 38.1 mm to (28.5, 5.00), turned to 180 degrees
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Connections:
- net A0: now also JP2.5; no longer JP2.2
- net A1: now also JP2.6; no longer JP2.3
- net A2: now also JP2.7; no longer JP2.4
- net A3: now also JP2.8; no longer JP2.5
- net A4: now also JP2.9; no longer JP2.6
- net A5: now also JP2.10; no longer JP2.7
- net AREF: now also JP2.11; no longer JP2.8
- net GND: no longer U1.EPAD
- net SPI_MISO: now also JP2.2; no longer JP2.11
- net SPI_MOSI: now also JP2.4; no longer JP2.10
- net SPI_SCK: now also JP2.3; no longer JP2.9
Routing:
- net VBUS: track 16.1 -> 47.2 mm, vias 3 -> 2
- net AREF: track 0.00 -> 26.6 mm
- net A4: track 0.00 -> 24.2 mm, vias 0 -> 1
- net A5: track 0.00 -> 23.6 mm
- net IRQ_LORA: track 0.00 -> 22.0 mm, vias 0 -> 1
- net A3: track 0.00 -> 21.4 mm, vias 0 -> 1
- net SPI_MOSI: track 0.00 -> 19.5 mm, vias 0 -> 1
- net A2: track 0.00 -> 17.9 mm, vias 0 -> 1
- net SPI_SCK: track 0.00 -> 17.8 mm, vias 0 -> 1
- net GND: track 31.5 -> 49.2 mm, vias 20 -> 27
- net SPI_MISO: track 0.00 -> 16.9 mm, vias 0 -> 1
- net A1: track 0.00 -> 16.1 mm, vias 0 -> 1
- net MISO_LORA: track 0.00 -> 13.1 mm, vias 0 -> 1
- net A0: track 0.00 -> 12.4 mm, vias 0 -> 1
- net VDDANA: track 0.00 -> 10.7 mm
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- added copper zone on layer 2, net +3V3

Commit message: layout_finish
Parts:
- moved R5 31.9 mm to (10.1, 13.3), flipped to the bottom
- moved R4 30.8 mm to (10.7, 12.2), flipped to the bottom
- moved C5 29.9 mm to (9.90, 11.1), flipped to the bottom, turned to 180 degrees
- moved U5 29.7 mm to (9.90, 8.80), flipped to the bottom, turned to 90 degrees
- moved C12 3.95 mm to (28.5, 13.0), turned to 0 degrees
- moved C8 3.80 mm to (12.6, 5.80), turned to 270 degrees
- moved C7 3.12 mm to (15.1, 17.9), flipped to the bottom, turned to 90 degrees
- moved L1 2.21 mm to (28.5, 14.8), turned to 180 degrees
Routing:
- net I2C_SCL: track 8.20 -> 55.6 mm, vias 0 -> 1
- net I2C_SDA: track 7.23 -> 48.9 mm, vias 0 -> 1
- net D10: track 3.08 -> 32.4 mm
- net D7: track 6.05 -> 30.4 mm, vias 0 -> 1
- net D6: track 4.78 -> 26.4 mm
- net D9: track 0.00 -> 17.9 mm, vias 0 -> 1
- net D5: track 0.00 -> 16.1 mm, vias 0 -> 1
- net D2: track 0.00 -> 13.3 mm, vias 0 -> 1
- net GND: track 49.2 -> 61.6 mm, vias 27 -> 31
- net +3V3: track 18.7 -> 29.0 mm, vias 5 -> 8
- net MOSI_LORA: track 0.00 -> 8.96 mm, vias 0 -> 1
- net CS_LORA: track 0.00 -> 5.30 mm, vias 0 -> 1
- net SCK_LORA: track 0.24 -> 5.24 mm, vias 0 -> 1
- net VDDANA: track 10.7 -> 8.74 mm
- net SPI_SCK: track 17.8 -> 18.4 mm
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- added copper zone on layer 1, net GND

Commit message: uodate
Routing:
- net GND: track 61.6 -> 56.3 mm, vias 31 -> 30
Changed lines of the file:
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@@
 <grid distance="0.1" unitdist="mm" unit="mm" style="lines" multiple="1" display="yes" altdistance="0.05" altunitdist="mm" altunit="mm"/>
 <layers>
-<layer number="1" name="Top" color="4" fill="1" visible="yes" active="yes"/>
+<layer number="1" name="Top" color="4" fill="1" visible="no" active="yes"/>
 <layer number="2" name="Route2" color="16" fill="1" visible="no" active="yes"/>
 <layer number="3" name="Route3" color="17" fill="1" visible="no" active="yes"/>
@@
 <layer number="14" name="Route14" color="22" fill="1" visible="no" active="no"/>
 <layer number="15" name="Route15" color="23" fill="1" visible="no" active="no"/>
-<layer number="16" name="Bottom" color="1" fill="1" visible="yes" active="yes"/>
-<layer number="17" name="Pads" color="2" fill="1" visible="yes" active="yes"/>
-<layer number="18" name="Vias" color="2" fill="1" visible="yes" active="yes"/>
-<layer number="19" name="Unrouted" color="6" fill="1" visible="yes" active="yes"/>
-<layer number="20" name="Dimension" color="24" fill="1" visible="yes" active="yes"/>
+<layer number="16" name="Bottom" color="1" fill="1" visible="no" active="yes"/>
+<layer number="17" name="Pads" color="2" fill="1" visible="no" active="yes"/>
+<layer number="18" name="Vias" color="2" fill="1" visible="no" active="yes"/>
+<layer number="19" name="Unrouted" color="6" fill="1" visible="no" active="yes"/>
+<layer number="20" name="Dimension" color="24" fill="1" visible="no" active="yes"/>
 <layer number="21" name="tPlace" color="7" fill="1" visible="yes" active="yes"/>
-<layer number="22" name="bPlace" color="7" fill="1" visible="yes" active="yes"/>
-<layer number="23" name="tOrigins" color="15" fill="1" visible="yes" active="yes"/>
-<layer number="24" name="bOrigins" color="15" fill="1" visible="yes" active="yes"/>
-<layer number="25" name="tNames" color="7" fill="1" visible="yes" active="yes"/>
-<layer number="26" name="bNames" color="7" fill="1" visible="yes" active="yes"/>
+<layer number="22" name="bPlace" color="7" fill="1" visible="no" active="yes"/>
+<layer number="23" name="tOrigins" color="15" fill="1" visible="no" active="yes"/>
+<layer number="24" name="bOrigins" color="15" fill="1" visible="no" active="yes"/>
+<layer number="25" name="tNames" color="7" fill="1" visible="no" active="yes"/>
+<layer number="26" name="bNames" color="7" fill="1" visible="no" active="yes"/>
 <layer number="27" name="tValues" color="7" fill="1" visible="no" active="yes"/>
 <layer number="28" name="bValues" color="7" fill="1" visible="no" active="yes"/>
@@
 <layer number="37" name="tTest" color="7" fill="1" visible="no" active="yes"/>
 <layer number="38" name="bTest" color="7" fill="1" visible="no" active="yes"/>
-<layer number="39" name="tKeepout" color="4" fill="11" visible="yes" active="yes"/>
-<layer number="40" name="bKeepout" color="1" fill="11" visible="yes" active="yes"/>
-<layer number="41" name="tRestrict" color="4" fill="10" visible="yes" active="yes"/>
-<layer number="42" name="bRestrict" color="1" fill="10" visible="yes" active="yes"/>
+<layer number="39" name="tKeepout" color="4" fill="11" visible="no" active="yes"/>
+<layer number="40" name="bKeepout" color="1" fill="11" visible="no" active="yes"/>
+<layer number="41" name="tRestrict" color="4" fill="10" visible="no" active="yes"/>
+<layer number="42" name="bRestrict" color="1" fill="10" visible="no" active="yes"/>
 <layer number="43" name="vRestrict" color="2" fill="10" visible="no" active="yes"/>
 <layer number="44" name="Drills" color="7" fill="1" visible="no" active="yes"/>
@@
 <layer number="49" name="Reference" color="7" fill="1" visible="no" active="yes"/>
 <layer number="50" name="dxf" color="7" fill="1" visible="no" active="yes"/>
-<layer number="51" name="tDocu" color="7" fill="1" visible="yes" active="yes"/>
-<layer number="52" name="bDocu" color="7" fill="1" visible="yes" active="yes"/>
+<layer number="51" name="tDocu" color="7" fill="1" visible="no" active="yes"/>
+<layer number="52" name="bDocu" color="7" fill="1" visible="no" active="yes"/>
 <layer number="53" name="tGND_GNDA" color="7" fill="9" visible="no" active="no"/>
 <layer number="54" name="bGND_GNDA" color="1" fill="9" visible="no" active="no"/>
@@
 <contactref element="C13" pad="2"/>
 <contactref element="C15" pad="2"/>
-<contactref element="R7" pad="2"/>
-<contactref element="U4" pad="2"/>
 <contactref element="C16" pad="2"/>
 <contactref element="C17" pad="2"/>
@@
 <wire x1="4.5" y1="4.4" x2="4.05" y2="4.85" width="0.5" layer="1"/>
 <wire x1="4.05" y1="4.85" x2="4.05" y2="6" width="0.5" layer="1"/>
-<wire x1="8.9" y1="18.5954" x2="8.9" y2="19.8" width="0.4" layer="16"/>
-<via x="8.9" y="19.8" extent="1-16" drill="0.4"/>
 <wire x1="13.15" y1="17.6" x2="12.85" y2="17.9" width="0.4" layer="16"/>
 <wire x1="12.85" y1="17.9" x2="12.85" y2="19.65" width="0.4" layer="16"/>
@@
 <wire x1="12.45" y1="21.05" x2="11" y2="21.05" width="0.4" layer="16"/>
 <wire x1="12.85" y1="20.65" x2="12.45" y2="21.05" width="0.4" layer="16"/>
-<wire x1="8.5206" y1="17.0206" x2="6.2206" y2="17.0206" width="0.254" layer="16"/>
-<wire x1="6.2" y1="17" x2="6.2206" y2="17.0206" width="0.254" layer="16"/>
-<wire x1="8.5206" y1="17.0206" x2="8.9" y2="17.4" width="0.254" layer="16"/>
-<wire x1="8.9" y1="17.4" x2="8.9" y2="18.5954" width="0.254" layer="16"/>
 <wire x1="12.5" y1="1.55" x2="11.1" y2="1.55" width="0.4" layer="16"/>
 <wire x1="11.1" y1="1.55" x2="10.9" y2="1.35" width="0.4" layer="16"/>
@@
 <vertex x="51" y="23"/>
 </polygon>
+<contactref element="R7" pad="2"/>
+<contactref element="U4" pad="2"/>
 </signal>
 <signal name="XIN32">

Commit message: update
Parts:
- removed H3, H4: MOUNT-HOLE2.5, Adafruit Feather M0 RFMxx:MICROBUILDER_MOUNTINGHOLE_2.5_PLATED
Other:
- board text added: "3V3"
- board text added: "A0"
- board text added: "A1"
- board text added: "A2"
- board text added: "A3"
- board text added: "A4"
- board text added: "A5"
- board text added: "AREF"
- board text added: "D0"
- board text added: "D1"
- board text added: "D10"
- board text added: "D2"
- board text added: "D5"
- board text added: "D6"
- board text added: "D7"
- board text added: "D9"
- board text added: "GND"
- board text added: "MISO"
- board text added: "MOSI"
- board text added: "SCK"
- board text added: "SCL"
- board text added: "SDA"
- board text added: "VBUS"

Commit message: update
Parts:
- C10: value 1µ -> 1u
Changed lines of the file:
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@@
 <attribute name="VALUE" x="29.135" y="6.905" size="1.27" layer="27" rot="R180"/>
 </element>
-<element name="C10" library="rcl" library_urn="urn:adsk.eagle:library:334" package="C0402" package3d_urn="urn:adsk.eagle:package:23626/2" value="1µ" x="16.8" y="5.2" smashed="yes" rot="R180">
+<element name="C10" library="rcl" library_urn="urn:adsk.eagle:library:334" package="C0402" package3d_urn="urn:adsk.eagle:package:23626/2" value="1u" x="16.8" y="5.2" smashed="yes" rot="R180">
 <attribute name="NAME" x="17.435" y="4.565" size="1.27" layer="25" rot="R180"/>
 <attribute name="POPULARITY" value="18" x="-30.19" y="73.78" size="1.778" layer="27" rot="R180" display="off"/>
